File: TransistorTester/TransistorTester.kicad_sch (KiCad schematic)
At the start: 19 parts, among them J1 Conn_01x02, J10 Conn_01x03_Pin, J2 Conn_01x02, J3 Conn_01x02, J4 Conn_01x03_Pin, J5 Conn_01x03_Pin, J6 Conn_01x03_Pin, J7 Conn_01x02, J8 Conn_01x03_Pin, J9 Conn_01x03_Pin

Commit message: fix resistors
Parts:
- added R4: 100, Resistor_SMD:R_0805_2012Metric_Pad1.20x1.40mm_HandSolder, symbol Device:R
- added RT4: 100, Resistor_THT:R_Axial_DIN0411_L9.9mm_D3.6mm_P12.70mm_Horizontal, symbol Device:R
- R1: value 50R -> 100
- RT1: value 50 -> 100
Connections:
- net GND: now also R4.1, RT4.1
- net at J2.2 (Pin_2), R1.2, R2.1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: now also R4.2, RT4.2
Other:
- note added: "All resistors are doubled : R* are SMD and RT* are THT (through hole technology). On the PCB, it will be possible to choice between SMD or THT as I have seen that made by others..."
- moved on the sheet: R2, RT2

Commit message: adapt to board
Parts:
- J10, J4, J5, J6, J8, J9: footprint Connector_PinHeader_2.54mm:PinHeader_1x03_P2.54mm_Vertical -> Connector_PinSocket_2.54mm:PinSocket_1x03_P2.54mm_Vertical
Connections:
- net at J2.2 (Pin_2), R1.2, R2.1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: no longer TP1.2
- net at J5.1 (Pin_1), J5.2 (Pin_2), J5.3 (Pin_3)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: now also TP1.2
Other:
- note added: "Transistors Tester / comparator"
Changed lines of the file:
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@@
+    (stroke (width 0) (type default))
+  )
+  (wire (pts (xy 106.68 76.2) (xy 106.68 85.09))
     (stroke (width 0) (type default))
   )
@@
     (stroke (width 0) (type default))
   )
-  (wire (pts (xy 74.93 76.2) (xy 93.98 76.2))
-    (stroke (width 0) (type default))
-  )
-  (wire (pts (xy 93.98 76.2) (xy 93.98 85.09))
+  (wire (pts (xy 74.93 76.2) (xy 106.68 76.2))
     (stroke (width 0) (type default))
   )
@@
   (wire (pts (xy 119.38 68.58) (xy 138.43 68.58))
     (stroke (width 0) (type default))
+  )
+  (text "   Transistors\nTester / comparator" (at 119.38 113.03 0)
+    (effects (font (size 1.27 1.27)) (justify left bottom))
   )
   (text "All resistors are doubled : R* are SMD and RT* are\nTHT (through hole technology). On the PCB, it will be\npossible to choice between SMD or THT as I have seen\nthat made by others..."
@@
       (effects (font (size 1.27 1.27)))
     )
-    (property "Footprint" "Connector_PinHeader_2.54mm:PinHeader_1x03_P2.54mm_Vertical" (at 116.84 77.47 0)
+    (property "Footprint" "Connector_PinSocket_2.54mm:PinSocket_1x03_P2.54mm_Vertical" (at 116.84 77.47 0)
       (effects (font (size 1.27 1.27)) hide)
     )
@@
       (effects (font (size 1.27 1.27)))
     )
-    (property "Footprint" "Connector_PinHeader_2.54mm:PinHeader_1x03_P2.54mm_Vertical" (at 149.86 77.47 0)
+    (property "Footprint" "Connector_PinSocket_2.54mm:PinSocket_1x03_P2.54mm_Vertical" (at 149.86 77.47 0)
       (effects (font (size 1.27 1.27)) hide)
     )
@@
       (effects (font (size 1.27 1.27)))
     )
-    (property "Footprint" "Connector_PinHeader_2.54mm:PinHeader_1x03_P2.54mm_Vertical" (at 149.86 60.96 0)
+    (property "Footprint" "Connector_PinSocket_2.54mm:PinSocket_1x03_P2.54mm_Vertical" (at 149.86 60.96 0)
       (effects (font (size 1.27 1.27)) hide)
     )
@@
       (effects (font (size 1.27 1.27)))
     )
-    (property "Footprint" "Connector_PinHeader_2.54mm:PinHeader_1x03_P2.54mm_Vertical" (at 116.84 90.17 0)
+    (property "Footprint" "Connector_PinSocket_2.54mm:PinSocket_1x03_P2.54mm_Vertical" (at 116.84 90.17 0)
       (effects (font (size 1.27 1.27)) hide)
     )
@@
       (effects (font (size 1.27 1.27)))
     )
-    (property "Footprint" "Connector_PinHeader_2.54mm:PinHeader_1x03_P2.54mm_Vertical" (at 116.84 60.96 0)
+    (property "Footprint" "Connector_PinSocket_2.54mm:PinSocket_1x03_P2.54mm_Vertical" (at 116.84 60.96 0)
       (effects (font (size 1.27 1.27)) hide)
     )
@@
       (effects (font (size 1.27 1.27)))
     )
-    (property "Footprint" "Connector_PinHeader_2.54mm:PinHeader_1x03_P2.54mm_Vertical" (at 149.86 90.17 0)
-      (effects (font (size 1.27 1.27)) hide)
-    )
+    (property "Footprint" "Connector_PinSocket_2.54mm:PinSocket_1x03_P2.54mm_Vertical" (at 149.86 90.17 0)
+      (effects (font (size 1.27 1.27)) hide)
+    )
