File: TransistorCurveTracer/TransistorCurveTracer.kicad_pcb (KiCad board)
At the start: 2 copper layers, 46 parts, among them J1 Conn_01x04_Pin, J2 Conn_01x04_Pin, J3 Conn_01x04_Pin, J4 Conn_01x04_Pin, J5 Conn_01x05_Pin, J6 Conn_01x05_Pin, Q1 BC547, Q2 BC547, Q3 BC547, Q4 2N2907, Q5 2N2907, Q6 DUT, U1 NE555P, U2 MCP601-xP, U3 MCP601-xP, U4 MCP601-xP

Commit message: 5 modules
Parts:
- removed the C2 at (52.4, 38.6)
- removed the C3 at (45.3, 51.6)
- removed the C4 at (33.9, 42.9)
- removed the D3 at (28.4, 50.0)
- removed the D4 at (28.4, 43.1)
- removed the J1 at (35.8, 25.4)
- removed J6: Conn_01x05_Pin, Connector_PinHeader_2.54mm:PinHeader_1x05_P2.54mm_Vertical
- removed the Q1 at (101.9, 25.7)
- removed the R10 at (95.0, 24.1)
- removed the R8 at (28.3, 35.6)
- removed the R9 at (28.3, 30.3)
- removed the U1 at (38.1, 38.1)
- added C1: 10n, Capacitor_THT:C_Disc_D7.5mm_W2.5mm_P5.00mm, F.Cu at (-9.24, 56.8)
- added C1: 10n, Capacitor_THT:C_Disc_D7.5mm_W2.5mm_P5.00mm, F.Cu at (27.9, 86.3)
- added C2: 10n, Capacitor_THT:C_Disc_D7.5mm_W2.5mm_P5.00mm, F.Cu at (-9.24, 60.8)
- added C2: 10n, Capacitor_THT:C_Disc_D7.5mm_W2.5mm_P5.00mm, F.Cu at (30.5, 53.3)
- added C4: 47u, Capacitor_THT:CP_Radial_D13.0mm_P5.00mm, F.Cu at (-6.13, 47.5)
- added C4: 47u, Capacitor_THT:CP_Radial_D13.0mm_P5.00mm, F.Cu at (25.5, 27.9)
- added D1: 1N4148, Diode_THT:D_DO-15_P15.24mm_Horizontal, F.Cu at (-28.5, 25.4)
- added D1: 1N4148, Diode_THT:D_DO-15_P15.24mm_Horizontal, F.Cu at (17.8, 71.1)
- added D2: 1N4148, Diode_THT:D_DO-15_P15.24mm_Horizontal, F.Cu at (22.9, 86.4)
- added D2: 1N4148, Diode_THT:D_DO-15_P15.24mm_Horizontal, F.Cu at (-28.5, 30.6)
- added J1: Conn_01x06_Pin, Connector_PinHeader_2.54mm:PinHeader_1x06_P2.54mm_Horizontal, F.Cu at (17.8, 17.8)
- added J1: Conn_01x06_Pin, Connector_PinHeader_2.54mm:PinHeader_1x06_P2.54mm_Horizontal, F.Cu at (-8.94, 25.2)
- added Q2: BC547, Package_TO_SOT_THT:TO-92_Inline, F.Cu at (27.9, 43.2)
- added Q2: BC547, Package_TO_SOT_THT:TO-92_Inline, F.Cu at (-0.23, 58.0)
- added R1: 39k, Resistor_THT:R_Axial_DIN0411_L9.9mm_D3.6mm_P15.24mm_Horizontal, F.Cu at (-28.5, 35.7)
- added R1: 39k, Resistor_THT:R_Axial_DIN0411_L9.9mm_D3.6mm_P15.24mm_Horizontal, F.Cu at (17.5, 50.8)
- added R3: 4.7k, Resistor_THT:R_Axial_DIN0411_L9.9mm_D3.6mm_P15.24mm_Horizontal, F.Cu at (-28.5, 40.9)
- added R3: 4.7k, Resistor_THT:R_Axial_DIN0411_L9.9mm_D3.6mm_P15.24mm_Horizontal, F.Cu at (17.5, 32.5)
- added R7: 10k, Resistor_THT:R_Axial_DIN0411_L9.9mm_D3.6mm_P15.24mm_Horizontal, F.Cu at (22.9, 53.3)
- added R7: 10k, Resistor_THT:R_Axial_DIN0411_L9.9mm_D3.6mm_P15.24mm_Horizontal, F.Cu at (-28.5, 46.0)
- added RV1: 0-5k, Connector_PinSocket_2.54mm:PinSocket_1x03_P2.54mm_Vertical, F.Cu at (221.7, 45.0)
- added U1: NE555P, Package_DIP:DIP-8_W7.62mm, F.Cu at (23.1, 58.4)
- added U1: NE555P, Package_DIP:DIP-8_W7.62mm, F.Cu at (-28.8, 50.7)
- C3: renamed from C6; footprint Capacitor_SMD:C_1206_3216Metric_Pad1.33x1.80mm_HandSolder -> Capacitor_THT:C_Disc_D7.5mm_W2.5mm_P5.00mm
- C5: renamed from C1; footprint Capacitor_SMD:C_0805_2012Metric_Pad1.18x1.45mm_HandSolder -> Capacitor_THT:C_Disc_D7.5mm_W2.5mm_P5.00mm
- C6: renamed from C5; footprint Capacitor_SMD:C_0805_2012Metric_Pad1.18x1.45mm_HandSolder -> Capacitor_THT:C_Disc_D7.5mm_W2.5mm_P5.00mm; moved to F.Cu
- D3: renamed from D1; footprint Diode_SMD:D_1812_4532Metric_Pad1.30x3.40mm_HandSolder -> Diode_THT:D_DO-15_P15.24mm_Horizontal
- D4: renamed from D2; footprint Diode_SMD:D_1812_4532Metric_Pad1.30x3.40mm_HandSolder -> Diode_THT:D_DO-15_P15.24mm_Horizontal
- J2, J3, J4: value Conn_01x04_Pin -> Conn_01x06_Pin; footprint Connector_PinHeader_2.54mm:PinHeader_1x04_P2.54mm_Vertical -> Connector_PinHeader_2.54mm:PinHeader_1x06_P2.54mm_Horizontal
- J5: value Conn_01x05_Pin -> Conn_01x06_Pin; footprint Connector_PinHeader_2.54mm:PinHeader_1x05_P2.54mm_Vertical -> Connector_PinHeader_2.54mm:PinHeader_1x06_P2.54mm_Horizontal
- R10: renamed from R19; footprint Resistor_SMD:R_1206_3216Metric_Pad1.30x1.75mm_HandSolder -> Resistor_THT:R_Axial_DIN0411_L9.9mm_D3.6mm_P15.24mm_Horizontal
- R11: renamed from R4; value 2.2k -> 1k; footprint Resistor_SMD:R_1206_3216Metric_Pad1.30x1.75mm_HandSolder -> Resistor_THT:R_Axial_DIN0411_L9.9mm_D3.6mm_P15.24mm_Horizontal
- R12: renamed from R5; footprint Resistor_THT:R_Axial_DIN0207_L6.3mm_D2.5mm_P2.54mm_Vertical -> Resistor_THT:R_Axial_DIN0411_L9.9mm_D3.6mm_P15.24mm_Horizontal
- R13: renamed from R3; footprint Resistor_THT:R_Axial_DIN0207_L6.3mm_D2.5mm_P2.54mm_Vertical -> Resistor_THT:R_Axial_DIN0411_L9.9mm_D3.6mm_P15.24mm_Horizontal
- R14: renamed from R7; footprint Resistor_SMD:R_1206_3216Metric_Pad1.30x1.75mm_HandSolder -> Resistor_THT:R_Axial_DIN0411_L9.9mm_D3.6mm_P15.24mm_Horizontal
- R15: renamed from R6; footprint Resistor_SMD:R_1206_3216Metric_Pad1.30x1.75mm_HandSolder -> Resistor_THT:R_Axial_DIN0411_L9.9mm_D3.6mm_P15.24mm_Horizontal
- R16: renamed from R20; footprint Resistor_SMD:R_1206_3216Metric_Pad1.30x1.75mm_HandSolder -> Resistor_THT:R_Axial_DIN0411_L9.9mm_D3.6mm_P15.24mm_Horizontal
- R17: renamed from R12; footprint Resistor_SMD:R_1206_3216Metric_Pad1.30x1.75mm_HandSolder -> Resistor_THT:R_Axial_DIN0411_L9.9mm_D3.6mm_P15.24mm_Horizontal
- R18: renamed from R11; footprint Resistor_SMD:R_1206_3216Metric_Pad1.30x1.75mm_HandSolder -> Resistor_THT:R_Axial_DIN0411_L9.9mm_D3.6mm_P15.24mm_Horizontal; moved to F.Cu
- R19: renamed from R13; footprint Resistor_SMD:R_1206_3216Metric_Pad1.30x1.75mm_HandSolder -> Resistor_THT:R_Axial_DIN0411_L9.9mm_D3.6mm_P15.24mm_Horizontal
- R2: renamed from R16; footprint Resistor_SMD:R_1206_3216Metric_Pad1.30x1.75mm_HandSolder -> Resistor_THT:R_Axial_DIN0411_L9.9mm_D3.6mm_P15.24mm_Horizontal
- R20: renamed from R14; footprint Resistor_SMD:R_1206_3216Metric_Pad1.30x1.75mm_HandSolder -> Resistor_THT:R_Axial_DIN0411_L9.9mm_D3.6mm_P15.24mm_Horizontal; moved to F.Cu
- R4: renamed from R15; footprint Resistor_SMD:R_1206_3216Metric_Pad1.30x1.75mm_HandSolder -> Resistor_THT:R_Axial_DIN0411_L9.9mm_D3.6mm_P15.24mm_Horizontal
- R5: renamed from R17; footprint Resistor_SMD:R_1206_3216Metric_Pad1.30x1.75mm_HandSolder -> Resistor_THT:R_Axial_DIN0411_L9.9mm_D3.6mm_P15.24mm_Horizontal
- R6: renamed from R18; footprint Resistor_SMD:R_1206_3216Metric_Pad1.30x1.75mm_HandSolder -> Resistor_THT:R_Axial_DIN0411_L9.9mm_D3.6mm_P15.24mm_Horizontal
- R8: renamed from R1; footprint Resistor_SMD:R_1206_3216Metric_Pad1.30x1.75mm_HandSolder -> Resistor_THT:R_Axial_DIN0411_L9.9mm_D3.6mm_P15.24mm_Horizontal
- R9: renamed from R2; footprint Resistor_SMD:R_1206_3216Metric_Pad1.30x1.75mm_HandSolder -> Resistor_THT:R_Axial_DIN0411_L9.9mm_D3.6mm_P15.24mm_Horizontal
- moved J2 187.7 mm to (223.5, 15.2)
- moved R17 179.2 mm to (277.1, 48.3)
- moved R19 175.0 mm to (277.1, 29.5)
- moved R18 165.6 mm to (258.8, 43.9)
- moved U4 161.9 mm to (265.2, 31.0), turned to 0 degrees
- moved R20 158.0 mm to (267.5, 59.2), turned to 90 degrees
- moved C6 151.1 mm to (263.1, 44.0), turned to -90 degrees
- moved Q6 144.6 mm to (258.8, 38.0), turned to 0 degrees
- moved R8 141.0 mm to (243.6, 40.6), turned to 90 degrees
- moved U3 128.5 mm to (230.6, 23.1), turned to 0 degrees
- moved R9 124.5 mm to (243.6, 45.2), turned to -90 degrees
- moved R13 119.9 mm to (236.7, 45.2), turned to -90 degrees
- moved R14 116.9 mm to (228.6, 66.0)
- moved R15 115.8 mm to (223.3, 34.5)
- moved R11 115.7 mm to (222.2, 66.5), turned to 90 degrees
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- renumbered Q3 to Q1, Q6 to Q3, Q2 to Q6, U4 to U2, U2 to U4
Connections:
- C6 pad 1: /ResetStairStep -> Net-(Q6-C)
- J2 pad 2: GND -> /SignalReset
- J2 pad 4: /Reset555 -> /StairStep
- J3 pad 2: GND -> /SignalReset
- J3 pad 3: /ResetStairStep -> /Out555
- J3 pad 4: /Reset555 -> /StairStep
- J4 pad 2: GND -> /SignalReset
- J4 pad 4: /SawTooth -> /StairStep
- J5 pad 2: GND -> /SignalReset
- J5 pad 4: /ResetStairStep -> /StairStep
- J5 pad 5: /StairStep -> /SawTooth
- Q6 pad 1: /ResetStairStep -> Net-(Q6-C)
- Q6 pad 2: /Pulse1 -> /SignalReset
- R11 pad 2: Net-(R3-Pad2) -> Net-(R11-Pad2)
- R12 pad 2: Net-(R3-Pad2) -> Net-(R12-Pad2)
- R13 pad 2: Net-(R3-Pad2) -> Net-(R12-Pad2)
- R14 pad 1: Net-(R3-Pad2) -> Net-(R12-Pad2)
- R15 pad 1: Net-(R3-Pad2) -> Net-(R12-Pad2)
- R15 pad 2: /Pulse1 -> /SignalReset
- R18 pad 1: /ResetStairStep -> Net-(Q6-C)
- R20 pad 2: /ResetStairStep -> Net-(Q6-C)
- U3 pad 6: Net-(R3-Pad2) -> Net-(R12-Pad2)
- U4 pad 3: /ResetStairStep -> Net-(Q6-C)
Routing:
- net /ResetStairStep: track 110.3 -> 0.00 mm, vias 2 -> 0
- net Net-(R12-Pad2): track 0.00 -> 87.3 mm
- net /Out555: track 10.3 -> 73.5 mm, vias 0 -> 3
- net Net-(R3-Pad2): track 62.8 -> 0.00 mm, vias 2 -> 0
- net Net-(D3-K): track 24.5 -> 76.7 mm, vias 1 -> 0
- net /StairStep: track 49.3 -> 0.35 mm
- net Net-(D1-A): track 0.00 -> 48.5 mm
- net Net-(D2-A): track 0.00 -> 41.0 mm
- net Net-(U3-+): track 0.00 -> 35.7 mm
- net /SignalReset: track 0.00 -> 34.3 mm
- net (no net): track 24.1 -> 0.00 mm
- net /Pulse1: track 21.4 -> 0.00 mm
- net Net-(U4--): track 16.5 -> 0.00 mm
- net /X: track 61.4 -> 46.8 mm
- net Net-(U1-CV): track 0.00 -> 13.8 mm
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Other:
- board text added: "SignalReset"
- board text removed: "NE555"
- board text removed: "ResertNE555 + Reset StairStep"
